Commit message: Add MoveIt configuration and launch files for davinci_arm
- Implemented ValueTile widget for displaying values with labels and units.
- Created .gitignore for hardware control package.
- Added MoveIt setup assistant configuration for davinci_arm.
- Developed CMakeLists.txt for building the MoveIt configuration package.
- Defined SRDF and URDF files for the davinci_arm robot model.
- Configured joint limits, kinematics, and MoveIt controllers.
- Created launch files for integrating Gazebo with MoveIt and RViz.
- Added RViz configuration for visualizing the robot and motion planning.
- Established warehouse database launch for storing planning data.
- Updated package.xml with dependencies and metadata for the MoveIt configuration package.

File: davinci_arm_description/models/davinci_arm_v3/urdf/davinci_arm.urdf.xacro (robot description, xacro)
@@ -29,4 +29,6 @@
     <!-- Joint between wrist and end effector -->
     <xacro:joint_module joint_name="end_effector_link_joint" parent="wrist_link" child="end_effector_link" xyz="-0.0430 0.0000 -0.0405" rpy="3.14159 -1.5708 0.0000" axis="0.0000 0.0000 1.0000"/>
+    <!-- Joint between end effector and marker -->
+    <xacro:link_module link_name="marker_link"/>
     <!-- Gazebo materials -->
     <xacro:include filename="$(find davinci_arm_gazebo_bridge)/urdf/gazebo_materials_support.xacro"/>

File: davinci_arm_description/models/davinci_arm_v3/urdf/davinci_arm_helpers.xacro (robot description, xacro)
@@ -22,4 +22,13 @@
         <material name="cad_cyan">
             <color rgba="0.0 0.72549 1.0 1.0"/>
+        </material>
+        <material name="marker_red">
+            <color rgba="0.85 0.05 0.05 1.0"/>
+        </material>
+        <material name="marker_white">
+            <color rgba="0.96 0.96 0.96 1.0"/>
+        </material>
+        <material name="marker_light_gray">
+            <color rgba="0.82 0.82 0.82 1.0"/>
         </material>
     </xacro:macro>
@@ -83,4 +92,9 @@
             <xacro:collision_mesh_component collision_name="end_effector_link_tool_holder_collision" mesh_file="tool_holder" xyz="-0.053 0 -0.0405" rpy="3.14159 -0.992087 -1.5708"/>
         </xacro:if>
+        <xacro:if value="${link_name == 'marker_link'}">
+            <xacro:collision_mesh_component collision_name="marker_body_collision" mesh_file="ExpoUltraFineBody" xyz="0 0 0" rpy="0 0 0"/>
+            <xacro:collision_mesh_component collision_name="marker_tip_base_collision" mesh_file="ExpoUltraFineTipBase" xyz="0 0 0" rpy="0 0 0"/>
+            <xacro:collision_mesh_component collision_name="marker_tip_collision" mesh_file="ExpoUltraFineTip" xyz="0 0 0" rpy="0 0 0"/>
+        </xacro:if>
     </xacro:macro>
     <!-- Inertial parameters taken from YAML -->
@@ -133,4 +147,10 @@
             <xacro:mesh_component visual_name="end_effector_link_tool_holder" mesh_file="tool_holder" xyz="-0.053 0 -0.0405" rpy="3.14159 -0.992087 -1.5708" material_name="cad_light_blue"/>
         </xacro:if>
+        <xacro:if value="${link_name == 'marker_link'}">
+            <xacro:mesh_component visual_name="marker_body_visual" mesh_file="ExpoUltraFineBody" xyz="0 0 0" rpy="0 0 0" material_name="marker_white"/>
+            <xacro:mesh_component visual_name="marker_tip_base_visual" mesh_file="ExpoUltraFineTipBase" xyz="0 0 0" rpy="0 0 0" material_name="marker_light_gray"/>
+            <xacro:mesh_component visual_name="marker_tip_visual" mesh_file="ExpoUltraFineTip" xyz="0 0 0" rpy="0 0 0" material_name="marker_red"/>
+            <xacro:mesh_component visual_name="marker_logo_visual" mesh_file="ExpoUltraFineBrandLogoProjection037" xyz="0 0 0" rpy="0 0 0" material_name="marker_red"/>
+        </xacro:if>
     </xacro:macro>
     <!-- Complete logical link -->
@@ -142,4 +162,9 @@
         </link>
     </xacro:macro>
+    <joint name="marker_link_joint" type="fixed">
+        <parent link="end_effector_link"/>
+        <child link="marker_link"/>
+        <origin xyz="-0.063 0.000 -0.0405" rpy="3.14159 -0.992087 -1.5708"/>
+    </joint>
     <!-- Revolute joint parameters taken from YAML -->
     <xacro:macro name="joint_module" params="joint_name parent child xyz rpy axis">

File: davinci_arm_gazebo_bridge/urdf/gazebo_materials_support.xacro (robot description, xacro)
@@ -48,4 +48,9 @@
         <xacro:gazebo_visual_material link_name="end_effector_link" visual_name="end_effector_link_size_0_flange" ambient="0.101961 0.101961 0.101961 1.0" diffuse="0.101961 0.101961 0.101961 1.0"/>
         <xacro:gazebo_visual_material link_name="end_effector_link" visual_name="end_effector_link_tool_holder" ambient="0.866667 0.909804 1.0 1.0" diffuse="0.866667 0.909804 1.0 1.0"/>
+        <!-- marker_link -->
+        <xacro:gazebo_visual_material link_name="marker_link" visual_name="marker_body_visual" ambient="0.96 0.96 0.96 1.0" diffuse="0.96 0.96 0.96 1.0"/>
+        <xacro:gazebo_visual_material link_name="marker_link" visual_name="marker_tip_base_visual" ambient="0.82 0.82 0.82 1.0" diffuse="0.82 0.82 0.82 1.0"/>
+        <xacro:gazebo_visual_material link_name="marker_link" visual_name="marker_tip_visual" ambient="0.85 0.05 0.05 1.0" diffuse="0.85 0.05 0.05 1.0" specular="0.25 0.05 0.05 1.0"/>
+        <xacro:gazebo_visual_material link_name="marker_link" visual_name="marker_logo_visual" ambient="0.85 0.05 0.05 1.0" diffuse="0.85 0.05 0.05 1.0" specular="0.25 0.05 0.05 1.0"/>
     </xacro:macro>
 </robot>

File: davinci_arm_gazebo_plugins/urdf/davinci_arm_control.xacro (robot description, xacro)
@@ -1,29 +1,32 @@
 <?xml version="1.0"?>
 <robot xmlns:xacro="http://www.ros.org/wiki/xacro" name="davinci_arm_control">
-    <ros2_control name="DaviniciArmSystem" type="system">
+    <ros2_control name="GazeboSimSystem" type="system">
+        <hardware>
+            <plugin>gz_ros2_control/GazeboSimSystem</plugin>
+        </hardware>
         <joint name="shoulder_link_joint">
+            <command_interface name="position"/>
             <state_interface name="position"/>
             <state_interface name="velocity"/>
-            <state_interface name="effort"/>
         </joint>
         <joint name="bicep_link_joint">
+            <command_interface name="position"/>
             <state_interface name="position"/>
             <state_interface name="velocity"/>
-            <state_interface name="effort"/>
         </joint>
         <joint name="arm_link_joint">
+            <command_interface name="position"/>
             <state_interface name="position"/>
             <state_interface name="velocity"/>
-            <state_interface name="effort"/>
         </joint>
         <joint name="wrist_link_joint">
+            <command_interface name="position"/>
             <state_interface name="position"/>
             <state_interface name="velocity"/>
-            <state_interface name="effort"/>
         </joint>
         <joint name="end_effector_link_joint">
+            <command_interface name="position"/>
             <state_interface name="position"/>
             <state_interface name="velocity"/>
-            <state_interface name="effort"/>
         </joint>
     </ros2_control>

File: davinci_arm_gazebo_plugins/urdf/davinci_arm_joint_position_model.xacro (robot description, xacro)
@@ -2,61 +2,64 @@
 <robot xmlns:xacro="http://www.ros.org/wiki/xacro">
     <gazebo>
-        <!-- Position controllers -->
         <plugin filename="gz-sim-joint-position-controller-system" name="gz::sim::systems::JointPositionController">
             <joint_name>shoulder_link_joint</joint_name>
             <topic>/davinci_arm/shoulder_cmd_pos</topic>
-            <p_gain>1.0</p_gain>
-            <i_gain>0.1</i_gain>
-            <d_gain>0.01</d_gain>
-            <i_max>1.0</i_max>
-            <i_min>-1.0</i_min>
+            <p_gain>20.0</p_gain>
+            <i_gain>0.5</i_gain>
+            <d_gain>1.0</d_gain>
+            <i_max>5.0</i_max>
+            <i_min>-5.0</i_min>
             <cmd_max>1000</cmd_max>
             <cmd_min>-1000</cmd_min>
+            <initial_position>0.0</initial_position>
         </plugin>
         <plugin filename="gz-sim-joint-position-controller-system" name="gz::sim::systems::JointPositionController">
             <joint_name>bicep_link_joint</joint_name>
             <topic>/davinci_arm/bicep_cmd_pos</topic>
-            <p_gain>1.0</p_gain>
-            <i_gain>0.1</i_gain>
-            <d_gain>0.01</d_gain>
-            <i_max>1.0</i_max>
-            <i_min>-1.0</i_min>
+            <p_gain>20.0</p_gain>
+            <i_gain>0.5</i_gain>
+            <d_gain>1.0</d_gain>
+            <i_max>5.0</i_max>
+            <i_min>-5.0</i_min>
             <cmd_max>1000</cmd_max>
             <cmd_min>-1000</cmd_min>
+            <initial_position>-1.5787</initial_position>
         </plugin>
         <plugin filename="gz-sim-joint-position-controller-system" name="gz::sim::systems::JointPositionController">
             <joint_name>arm_link_joint</joint_name>
             <topic>/davinci_arm/arm_cmd_pos</topic>
-            <p_gain>1.0</p_gain>
-            <i_gain>0.1</i_gain>
-            <d_gain>0.01</d_gain>
-            <i_max>1.0</i_max>
-            <i_min>-1.0</i_min>
+            <p_gain>20.0</p_gain>
+            <i_gain>0.5</i_gain>
+            <d_gain>1.0</d_gain>
+            <i_max>5.0</i_max>
+            <i_min>-5.0</i_min>
             <cmd_max>1000</cmd_max>
             <cmd_min>-1000</cmd_min>
+            <initial_position>0.0</initial_position>
         </plugin>
         <plugin filename="gz-sim-joint-position-controller-system" name="gz::sim::systems::JointPositionController">
             <joint_name>wrist_link_joint</joint_name>
             <topic>/davinci_arm/wrist_cmd_pos</topic>
-            <p_gain>1.0</p_gain>
-            <i_gain>0.1</i_gain>
-            <d_gain>0.01</d_gain>
-            <i_max>1.0</i_max>
-            <i_min>-1.0</i_min>
+            <p_gain>20.0</p_gain>
+            <i_gain>0.5</i_gain>
+            <d_gain>1.0</d_gain>
+            <i_max>5.0</i_max>
+            <i_min>-5.0</i_min>
             <cmd_max>1000</cmd_max>
             <cmd_min>-1000</cmd_min>
+            <initial_position>0.0</initial_position>
         </plugin>
         <plugin filename="gz-sim-joint-position-controller-system" name="gz::sim::systems::JointPositionController">
             <joint_name>end_effector_link_joint</joint_name>
             <topic>/davinci_arm/end_effector_cmd_pos</topic>
-            <p_gain>1.0</p_gain>
-            <i_gain>0.1</i_gain>
-            <d_gain>0.01</d_gain>
-            <i_max>1.0</i_max>
-            <i_min>-1.0</i_min>
+            <p_gain>20.0</p_gain>
+            <i_gain>0.5</i_gain>
+            <d_gain>1.0</d_gain>
+            <i_max>5.0</i_max>
+            <i_min>-5.0</i_min>
             <cmd_max>1000</cmd_max>
             <cmd_min>-1000</cmd_min>
+            <initial_position>1.5787</initial_position>
         </plugin>
-        <!-- Joint state publisher -->
         <plugin filename="gz-sim-joint-state-publisher-system" name="gz::sim::systems::JointStatePublisher">
             <topic>/davinci_arm/joint_states</topic>
